File: BNN/BNN_Power.kicad_sch (KiCad schematic)
At the start: 16 parts, among them J1 USB4110-GF-A, U1 AP2112K-3.3TRG1, U2 AP2112K-1.2TRG1

Commit message: Add files via upload
Connections:
- net +5V: no longer C5.2
- net at R4.2, U1.3 (EN): now also C5.2
Other:
- moved on the sheet: C1, C3, C5
Changed lines of the file:
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@@
 	(paper "A4")
 	(junction
+		(at 181.61 63.5)
+		(diameter 0)
+		(color 0 0 0 0)
+	)
+	(junction
 		(at 125.73 78.74)
 		(diameter 0)
@@
 	)
 	(junction
-		(at 234.95 105.41)
+		(at 167.64 48.26)
 		(diameter 0)
 		(color 0 0 0 0)
 	)
 	(junction
-		(at 171.45 48.26)
+		(at 234.95 105.41)
 		(diameter 0)
 		(color 0 0 0 0)
@@
 	)
 	(junction
-		(at 163.83 48.26)
+		(at 234.95 48.26)
 		(diameter 0)
 		(color 0 0 0 0)
 	)
 	(junction
-		(at 234.95 48.26)
+		(at 180.34 105.41)
 		(diameter 0)
 		(color 0 0 0 0)
 	)
 	(junction
-		(at 180.34 105.41)
+		(at 175.26 48.26)
 		(diameter 0)
 		(color 0 0 0 0)
@@
 	(wire
 		(pts
-			(xy 163.83 102.87) (xy 163.83 105.41)
+			(xy 181.61 63.5) (xy 181.61 66.04)
 		)
 		(stroke
@@
 	(wire
 		(pts
-			(xy 102.87 78.74) (xy 125.73 78.74)
+			(xy 163.83 102.87) (xy 163.83 105.41)
 		)
 		(stroke
@@
 	(wire
 		(pts
-			(xy 57.15 81.28) (xy 57.15 111.76)
+			(xy 102.87 78.74) (xy 125.73 78.74)
 		)
 		(stroke
@@
 	(wire
 		(pts
-			(xy 180.34 120.65) (xy 180.34 105.41)
+			(xy 57.15 81.28) (xy 57.15 111.76)
 		)
 		(stroke
@@
 	(wire
 		(pts
-			(xy 181.61 45.72) (xy 181.61 48.26)
+			(xy 180.34 120.65) (xy 180.34 105.41)
 		)
 		(stroke
@@
 	(wire
 		(pts
-			(xy 163.83 38.1) (xy 163.83 48.26)
+			(xy 167.64 38.1) (xy 167.64 48.26)
 		)
 		(stroke
@@
 	(wire
 		(pts
-			(xy 163.83 48.26) (xy 171.45 48.26)
+			(xy 234.95 102.87) (xy 234.95 105.41)
 		)
 		(stroke
@@
 	(wire
 		(pts
-			(xy 234.95 102.87) (xy 234.95 105.41)
+			(xy 57.15 111.76) (xy 125.73 111.76)
 		)
 		(stroke
@@
 	(wire
 		(pts
-			(xy 57.15 111.76) (xy 125.73 111.76)
+			(xy 123.19 57.15) (xy 123.19 76.2)
 		)
 		(stroke
@@
 	(wire
 		(pts
-			(xy 123.19 57.15) (xy 123.19 76.2)
+			(xy 255.27 102.87) (xy 255.27 105.41)
 		)
 		(stroke
@@
 	(wire
 		(pts
-			(xy 255.27 102.87) (xy 255.27 105.41)
+			(xy 104.14 101.6) (xy 45.72 101.6)
 		)
 		(stroke
@@
 	(wire
 		(pts
-			(xy 104.14 101.6) (xy 45.72 101.6)
+			(xy 158.75 45.72) (xy 158.75 48.26)
 		)
 		(stroke
@@
 	(wire
 		(pts
-			(xy 154.94 45.72) (xy 154.94 48.26)
+			(xy 85.09 170.18) (xy 85.09 175.26)
 		)
 		(stroke
@@
 	(wire
 		(pts
-			(xy 85.09 170.18) (xy 85.09 175.26)
+			(xy 180.34 102.87) (xy 180.34 105.41)
 		)
 		(stroke
@@
 	(wire
 		(pts
-			(xy 180.34 102.87) (xy 180.34 105.41)
+			(xy 167.64 48.26) (xy 175.26 48.26)
 		)
 		(stroke
@@
 	(wire
 		(pts
-			(xy 171.45 45.72) (xy 171.45 48.26)
+			(xy 175.26 45.72) (xy 175.26 48.26)
 		)
 		(stroke
@@
 	(wire
 		(pts
-			(xy 154.94 48.26) (xy 163.83 48.26)
+			(xy 158.75 48.26) (xy 167.64 48.26)
 		)
 		(stroke
@@
 	(wire
 		(pts
-			(xy 171.45 48.26) (xy 181.61 48.26)
+			(xy 104.14 86.36) (xy 104.14 101.6)
 		)
 		(stroke
@@
 	(wire
 		(pts
-			(xy 104.14 86.36) (xy 104.14 101.6)
+			(xy 175.26 48.26) (xy 181.61 48.26)
 		)
 		(stroke
@@
 	(symbol
 		(lib_id "power:GND")
-		(at 154.94 38.1 180)
+		(at 158.75 38.1 180)
 		(unit 1)
 		(exclude_from_sim no)
@@
 		(fields_autoplaced yes)
 		(property "Reference" "#PWR08"
-			(at 154.94 31.75 0)
+			(at 158.75 31.75 0)
 			(effects
 				(font
@@
 		)
 		(property "Value" "GND"
-			(at 154.94 33.02 0)
+			(at 158.75 33.02 0)
 			(effects
 				(font
@@
 		)
 		(property "Footprint" ""
-			(at 154.94 38.1 0)
+			(at 158.75 38.1 0)
 			(effects
 				(font
@@
 		)
 		(property "Datasheet" ""
-			(at 154.94 38.1 0)
+			(at 158.75 38.1 0)
 			(effects
 				(font
@@
 		)
 		(property "Description" ""
-			(at 154.94 38.1 0)
+			(at 158.75 38.1 0)
 			(effects
 				(font
@@
 	(symbol
 		(lib_id "1uF C:GCM188R71E105KA64D")
-		(at 181.61 38.1 270)
+		(at 181.61 73.66 90)
 		(unit 1)
 		(exclude_from_sim no)
@@
 		(dnp no)
 		(property "Reference" "C5"
-			(at 184.404 40.894 90)
+			(at 178.816 70.866 90)
 			(effects
 				(font
@@
 		)
 		(property "Value" "1uF"
-			(at 185.42 43.18 90)
+			(at 177.8 68.58 90)
 			(effects
 				(font
@@
 		)
 		(property "Footprint" "CAP_GCM188_MUR"
-			(at 181.61 38.1 0)
+			(at 181.61 73.66 0)
 			(effects
 				(font
@@
 		)
 		(property "Datasheet" "GCM188R71E105KA64D"
-			(at 181.61 38.1 0)
+			(at 181.61 73.66 0)
 			(effects
 				(font
@@
 		)
 		(property "Description" ""
-			(at 181.61 38.1 0)
+			(at 181.61 73.66 0)
 			(effects
 				(font
@@
 		)
 		(instances
-			(project ""
+			(project "BNN"
 				(path "/b0a0a466-abb8-40a5-aa14-c9034c337ed7/da5dddb6-27e9-4bf0-896e-d14bf9cd672c"
 					(reference "C5")
@@
 	(symbol
 		(lib_id "10uF C:GRM188R61E106KA73D")
-		(at 154.94 45.72 90)
+		(at 158.75 45.72 90)
 		(unit 1)
 		(exclude_from_sim no)
@@
 		(fields_autoplaced yes)
 		(property "Reference" "C1"
-			(at 158.75 41.2749 90)
+			(at 162.56 41.2749 90)
 			(effects
 				(font
@@
 		)
 		(property "Value" "10uF"
-			(at 158.75 43.18 90)
+			(at 162.56 43.18 90)
 			(effects
 				(font
@@
 		)
 		(property "Footprint" "ul_GRM188R61E106KA73D:CAP_GRM188_&plus_&slash_-0.2_MUR"
-			(at 154.94 45.72 0)
+			(at 158.75 45.72 0)
 			(effects
 				(font
@@
 		)
 		(property "Datasheet" "GRM188R61E106KA73D"
-			(at 154.94 45.72 0)
+			(at 158.75 45.72 0)
 			(effects
 				(font
@@
 		)
 		(property "Description" ""
-			(at 154.94 45.72 0)
+			(at 158.75 45.72 0)
 			(effects
 				(font
@@
 	(symbol
 		(lib_id "1uF C:GCM188R71E105KA64D")
-		(at 171.45 38.1 270)
+		(at 175.26 38.1 270)
 		(unit 1)
 		(exclude_from_sim no)
@@
 		(dnp no)
 		(property "Reference" "C3"
-			(at 174.244 40.894 90)
+			(at 178.054 40.894 90)
 			(effects
 				(font
@@
 		)
 		(property "Value" "1uF"
-			(at 175.26 43.18 90)
+			(at 179.07 43.18 90)
 			(effects
 				(font
@@
 		)
 		(property "Footprint" "CAP_GCM188_MUR"
-			(at 171.45 38.1 0)
+			(at 175.26 38.1 0)
 			(effects
 				(font
@@
 		)
 		(property "Datasheet" "GCM188R71E105KA64D"
-			(at 171.45 38.1 0)
+			(at 175.26 38.1 0)
 			(effects
 				(font
@@
 		)
 		(property "Description" ""
-			(at 171.45 38.1 0)
+			(at 175.26 38.1 0)
 			(effects
 				(font
@@
 	(symbol
 		(lib_id "power:GND")
-		(at 171.45 38.1 180)
+		(at 175.26 38.1 180)
 		(unit 1)
 		(exclude_from_sim no)
@@
 		(fields_autoplaced yes)
 		(property "Reference" "#PWR011"
-			(at 171.45 31.75 0)
+			(at 175.26 31.75 0)
 			(effects
 				(font
@@
 		)
 		(property "Value" "GND"
-			(at 171.45 33.02 0)
+			(at 175.26 33.02 0)
 			(effects
 				(font
@@
 		)
 		(property "Footprint" ""
-			(at 171.45 38.1 0)
+			(at 175.26 38.1 0)
 			(effects
 				(font
@@
 		)
 		(property "Datasheet" ""
-			(at 171.45 38.1 0)
+			(at 175.26 38.1 0)
 			(effects
 				(font
@@
 		)
 		(property "Description" ""
-			(at 171.45 38.1 0)
+			(at 175.26 38.1 0)
 			(effects
 				(font
@@
 	(symbol
 		(lib_id "power:GND")
-		(at 181.61 38.1 180)
+		(at 181.61 73.66 0)
 		(unit 1)
 		(exclude_from_sim no)
@@
 		(fields_autoplaced yes)
 		(property "Reference" "#PWR014"
-			(at 181.61 31.75 0)
+			(at 181.61 80.01 0)
 			(effects
 				(font
@@
 		)
 		(property "Value" "GND"
-			(at 181.61 33.02 0)
+			(at 184.15 74.9299 0)
 			(effects
 				(font
 					(size 1.27 1.27)
 				)
+				(justify left)
 			)
 		)
 		(property "Footprint" ""
-			(at 181.61 38.1 0)
+			(at 181.61 73.66 0)
 			(effects
 				(font
@@
 		)
 		(property "Datasheet" ""
-			(at 181.61 38.1 0)
+			(at 181.61 73.66 0)
 			(effects
 				(font
@@
 		)
 		(property "Description" ""
-			(at 181.61 38.1 0)
+			(at 181.61 73.66 0)
 			(effects
 				(font
@@
 	(symbol
 		(lib_id "power:+5V")
-		(at 163.83 38.1 0)
+		(at 167.64 38.1 0)
 		(unit 1)
 		(exclude_from_sim no)
@@
 		(fields_autoplaced yes)
 		(property "Reference" "#PWR09"
-			(at 163.83 41.91 0)
+			(at 167.64 41.91 0)
 			(effects
 				(font
@@
 		)
 		(property "Value" "+5V"
-			(at 163.83 33.02 0)
+			(at 167.64 33.02 0)
 			(effects
 				(font
@@
 		)
 		(property "Footprint" ""
-			(at 163.83 38.1 0)
+			(at 167.64 38.1 0)
 			(effects
 				(font
@@
 		)
 		(property "Datasheet" ""
-			(at 163.83 38.1 0)
+			(at 167.64 38.1 0)
 			(effects
 				(font
@@
 		)
 		(property "Description" "Power symbol creates a global label with name \"+5V\""
-			(at 163.83 38.1 0)
+			(at 167.64 38.1 0)
 			(effects
 				(font
