File: BNN/BNN.kicad_pcb (KiCad board)
At the start: 2 copper layers, 60.8 x 52.7 mm, 69 parts, among them J1 USB4110-GF-A, J2 DEBUG, J3 Conn_01x20, J4 Conn_01x12, J5 Conn_01x20, U1 AP2112K-3.3TRG1, U2 AP2112K-1.2TRG1, U3 SC09147, U4 W25Q32JWSSIQ, U5 W25Q32JWSSIQ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

Commit message: Add files via upload
Parts:
- moved C5 4.27 mm to (151.0, 84.9)
- moved C1 2.13 mm to (155.3, 84.9)
- moved C3 2.13 mm to (153.2, 85.0)
Connections:
- C5 pad 2: +5V -> Net-(U1-EN)
Routing:
- net Net-(U1-EN): track 2.23 -> 4.32 mm
- net +5V: track 146.7 -> 148.5 mm

Commit message: Add files via upload
Routing:
- net /iCE40UP5K/SPI_SS: track 31.7 -> 34.1 mm
Changed lines of the file:
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@@
 			(plot_on_all_layers_selection 0x00000000_00000000_00000000_00000000)
 			(disableapertmacros no)
-			(usegerberextensions no)
+			(usegerberextensions yes)
 			(usegerberattributes yes)
 			(usegerberadvancedattributes yes)
@@
 			(outputformat 1)
 			(mirror no)
-			(drillshape 1)
+			(drillshape 0)
 			(scaleselection 1)
-			(outputdirectory "")
+			(outputdirectory "./gerbers/")
 		)
 	)
@@
 	)
 	(segment
-		(start 158.4892 97.7561)
-		(end 156.7537 96.0206)
-		(width 0.2032)
-		(layer "F.Cu")
-		(net 1)
-	)
-	(segment
 		(start 136.226801 104.5464)
 		(end 136.226801 103.699383)
@@
 	)
 	(segment
+		(start 156.407206 96.2238)
+		(end 153.835502 96.2238)
+		(width 0.2032)
+		(layer "F.Cu")
+		(net 1)
+	)
+	(segment
 		(start 134.2268 104.5464)
 		(end 133.4232 103.7428)
@@
 	)
 	(segment
-		(start 139.1412 110.49)
-		(end 139.1412 108.350774)
-		(width 0.508)
+		(start 153.2486 96.810702)
+		(end 153.2486 96.9264)
+		(width 0.2032)
 		(layer "F.Cu")
 		(net 1)
 	)
 	(segment
-		(start 154.9298 96.2254)
-		(end 153.836164 96.2254)
-		(width 0.2)
+		(start 139.1412 110.49)
+		(end 139.1412 108.350774)
+		(width 0.508)
 		(layer "F.Cu")
 		(net 1)
@@
 	)
 	(segment
+		(start 158.696368 96.019)
+		(end 157.1617 96.019)
+		(width 0.2032)
+		(layer "F.Cu")
+		(net 1)
+	)
+	(segment
 		(start 134.177547 100.08895)
 		(end 134.177547 99.067868)
@@
 	)
 	(segment
+		(start 156.9569 96.2238)
+		(end 158.4892 97.7561)
+		(width 0.2)
+		(layer "F.Cu")
+		(net 1)
+	)
+	(segment
 		(start 129.3612 95.8596)
 		(end 128.685 95.1834)
@@
 	)
 	(segment
-		(start 153.836164 96.2254)
-		(end 153.2486 96.812964)
-		(width 0.2)
-		(layer "F.Cu")
-		(net 1)
-	)
-	(segment
 		(start 128.685 93.1758)
 		(end 126.4506 90.9414)
@@
 	)
 	(segment
+		(start 156.407206 96.2238)
+		(end 156.9569 96.2238)
+		(width 0.2)
+		(layer "F.Cu")
+		(net 1)
+	)
+	(segment
 		(start 134.4168 103.449701)
 		(end 134.4168 100.435901)
@@
 	)
 	(segment
+		(start 157.1617 96.019)
+		(end 156.9569 96.2238)
+		(width 0.2032)
+		(layer "F.Cu")
+		(net 1)
+	)
+	(segment
 		(start 139.2936 100.379101)
 		(end 139.2936 103.506501)
@@
 	)
 	(segment
-		(start 159.489201 97.7646)
-		(end 159.489201 96.811833)
-		(width 0.2032)
-		(layer "F.Cu")
-		(net 1)
-	)
-	(segment
 		(start 137.945898 99.24)
 		(end 138.583098 98.6028)
@@
 	)
 	(segment
-		(start 158.697968 96.0206)
-		(end 158.969167 96.291799)
-		(width 0.2)
-		(layer "F.Cu")
-		(net 1)
-	)
-	(segment
 		(start 158.895001 86.735699)
 		(end 155.1432 90.4875)
@@
 	)
 	(segment
-		(start 156.7537 96.0206)
-		(end 155.1346 96.0206)
-		(width 0.2)
-		(layer "F.Cu")
-		(net 1)
-	)
-	(segment
 		(start 154.8384 109.5756)
 		(end 154.8384 107.610199)
@@
 	)
 	(segment
-		(start 158.697968 96.0206)
-		(end 156.7537 96.0206)
-		(width 0.2)
-		(layer "F.Cu")
-		(net 1)
-	)
-	(segment
 		(start 139.2936 103.506501)
 		(end 139.529899 103.7428)
@@
 	)
 	(segment
+		(start 153.835502 96.2238)
+		(end 153.2486 96.810702)
+		(width 0.2032)
+		(layer "F.Cu")
+		(net 1)
+	)
+	(segment
 		(start 142.21 113.2332)
 		(end 139.2936 113.2332)
@@
 	)
 	(segment
-		(start 139.2936 113.2332)
-		(end 138.652402 112.592002)
-		(width 0.508)
+		(start 159.489201 96.811833)
+		(end 159.489201 97.7646)
+		(width 0.2032)
 		(layer "F.Cu")
 		(net 1)
 	)
 	(segment
-		(start 155.1346 96.0206)
-		(end 154.9298 96.2254)
-		(width 0.2)
+		(start 139.2936 113.2332)
+		(end 138.652402 112.592002)
+		(width 0.508)
 		(layer "F.Cu")
 		(net 1)
@@
 	)
 	(segment
-		(start 159.489201 96.811833)
-		(end 158.969167 96.291799)
-		(width 0.2032)
-		(layer "F.Cu")
-		(net 1)
-	)
-	(segment
 		(start 167.498 104.710799)
 		(end 165.475799 106.733)
@@
 	)
 	(segment
+		(start 158.696368 96.019)
+		(end 159.489201 96.811833)
+		(width 0.2032)
+		(layer "F.Cu")
+		(net 1)
+	)
+	(segment
 		(start 134.2268 104.5464)
 		(end 134.622601 104.5464)
@@
 	)
 	(segment
-		(start 148.1328 99.999048)
-		(end 148.1328 99.084653)
+		(start 152.180854 95.0366)
+		(end 152.790448 95.0366)
 		(width 0.1524)
 		(layer "F.Cu")
@@
 	)
 	(segment
-		(start 152.403653 94.8138)
-		(end 152.635782 94.8138)
+		(start 148.1328 99.999048)
+		(end 147.547848 100.584)
 		(width 0.1524)
 		(layer "F.Cu")
@@
 	)
 	(segment
-		(start 145.675204 100.584)
-		(end 147.547848 100.584)
+		(start 162.306 94.334899)
+		(end 162.306 92.8439)
 		(width 0.1524)
 		(layer "F.Cu")
@@
 	)
 	(segment
-		(start 147.547848 100.584)
-		(end 148.1328 99.999048)
+		(start 154.372449 93.4546)
+		(end 156.0576 93.4546)
 		(width 0.1524)
 		(layer "F.Cu")
@@
 	)
 	(segment
-		(start 162.306 94.334899)
-		(end 162.306 92.8439)
+		(start 152.790448 95.0366)
+		(end 154.372449 93.4546)
 		(width 0.1524)
 		(layer "F.Cu")
@@
 	)
 	(segment
-		(start 154.686 95.5214)
-		(end 158.4761 95.5214)
+		(start 148.1328 99.084654)
+		(end 152.180854 95.0366)
 		(width 0.1524)
 		(layer "F.Cu")
@@
 	)
 	(segment
-		(start 140.2304 100.9428)
-		(end 145.316404 100.9428)
+		(start 147.547848 100.584)
+		(end 145.675204 100.584)
 		(width 0.1524)
 		(layer "F.Cu")
@@
 	)
 	(segment
-		(start 148.1328 99.084653)
-		(end 152.403653 94.8138)
+		(start 158.4761 95.5214)
+		(end 156.0576 95.5214)
+		(width 0.1524)
+		(layer "F.Cu")
+		(net 84)
+	)
+	(segment
+		(start 148.1328 99.084654)
+		(end 148.1328 99.999048)
 		(width 0.1524)
 		(layer "F.Cu")
@@
 	(segment
 		(start 145.316404 100.9428)
-		(end 145.675204 100.584)
+		(end 140.2304 100.9428)
+		(width 0.1524)
+		(layer "F.Cu")
+		(net 84)
+	)
+	(segment
+		(start 145.675204 100.584)
+		(end 145.316404 100.9428)
 		(width 0.1524)
 		(layer "F.Cu")
@@
 	)
 	(via
-		(at 152.635782 94.8138)
+		(at 156.0576 95.5214)
 		(size 0.6)
 		(drill 0.3)
@@
 	)
 	(via
-		(at 154.686 95.5214)
+		(at 156.0576 93.4546)
 		(size 0.6)
 		(drill 0.3)
@@
 	)
 	(segment
-		(start 153.9784 94.8138)
-		(end 154.686 95.5214)
+		(start 156.0576 95.5214)
+		(end 156.0576 93.4546)
 		(width 0.1524)
 		(layer "B.Cu")
@@
 		(width 0.1524)
 		(layer "B.Cu")
-		(net 84)
-	)
-	(segment
-		(start 152.635782 94.8138)
-		(end 153.9784 94.8138)
-		(width 0.1524)
-		(layer "B.Cu")
